Commit message: Migrate ar_project to ROS 2 Jazzy and Gazebo Sim

File: description/camera.xacro (robot description, xacro)
@@ -23,7 +23,9 @@
         <sensor name="camera" type="camera">
             <pose>0 0 0 0 0 0</pose>
+            <always_on>true</always_on>
             <visualize>true</visualize>
             <update_rate>10</update_rate>
             <camera>
+                <camera_info_topic>camera/camera_info</camera_info_topic>
                 <horizontal_fov>1.089</horizontal_fov>
                 <image>
@@ -37,7 +39,6 @@
                 </clip>
             </camera>
-            <plugin name="camera_controller" filename="libgazebo_ros_camera.so">
-                <frame_name>camera_link_optical</frame_name>
-            </plugin>
+            <topic>camera/image_raw</topic>
+            <gz_frame_id>camera_link_optical</gz_frame_id>
         </sensor>
         <material>Gazebo/Red</material>

File: description/depth_camera.xacro (robot description, xacro)
@@ -23,23 +23,22 @@
         <sensor name="depth_camera" type="depth">
             <pose>0 0 0 0 0 0</pose>
+            <always_on>true</always_on>
             <visualize>true</visualize>
             <update_rate>10</update_rate>
+            <topic>depth_camera/depth/image_raw</topic>
+            <gz_frame_id>depth_camera_link_optical</gz_frame_id>
             <camera>
                 <horizontal_fov>1.089</horizontal_fov>
                 <image>
-                    <format>B8G8R8</format>
                     <width>640</width>
                     <height>480</height>
                 </image>
-                <clip>
-                    <near>0.05</near>
-                    <far>8.0</far>
-                </clip>
+                <depth_camera>
+                    <clip>
+                        <near>0.05</near>
+                        <far>8.0</far>
+                    </clip>
+                </depth_camera>
             </camera>
-            <plugin name="depth_camera_controller" filename="libgazebo_ros_camera.so">
-                <frame_name>camera_link_optical</frame_name>
-                <min_depth>0.1</min_depth>
-                <max_depth>100.0</max_depth>
-            </plugin>
         </sensor>
         <material>Gazebo/Red</material>

File: description/gazebo_control.xacro (robot description, xacro)
@@ -2,19 +2,25 @@
 <robot xmlns:xacro="http://www.ros.org/wiki/xacro">
     <gazebo>
-        <plugin name="diff_drive" filename="libgazebo_ros_diff_drive.so">
-            <!-- Wheel Information -->
+        <plugin name="gz::sim::systems::DiffDrive" filename="gz-sim-diff-drive-system">
             <left_joint>left_wheel_joint</left_joint>
             <right_joint>right_wheel_joint</right_joint>
             <wheel_separation>0.35</wheel_separation>
-            <wheel_diameter>0.1</wheel_diameter>
-            <!-- Limits -->
-            <max_wheel_torque>200</max_wheel_torque>
-            <max_wheel_acceleration>10.0</max_wheel_acceleration>
-            <!-- Output -->
-            <odometry_frame>odom</odometry_frame>
-            <robot_base_frame>base_link</robot_base_frame>
-            <publish_odom>true</publish_odom>
-            <publish_odom_tf>true</publish_odom_tf>
-            <publish_wheel_tf>true</publish_wheel_tf>
+            <wheel_radius>0.05</wheel_radius>
+            <max_linear_acceleration>0.5</max_linear_acceleration>
+            <min_linear_acceleration>-0.5</min_linear_acceleration>
+            <topic>cmd_vel</topic>
+            <odom_topic>odom</odom_topic>
+            <tf_topic>tf</tf_topic>
+            <frame_id>odom</frame_id>
+            <child_frame_id>base_link</child_frame_id>
+            <odom_publish_frequency>30</odom_publish_frequency>
+        </plugin>
+        <plugin
+            name="gz::sim::systems::JointStatePublisher"
+            filename="gz-sim-joint-state-publisher-system">
+            <joint_name>left_wheel_joint</joint_name>
+            <joint_name>right_wheel_joint</joint_name>
+            <topic>joint_states</topic>
+            <update_rate>30</update_rate>
         </plugin>
     </gazebo>

File: description/lidar.xacro (robot description, xacro)
@@ -23,8 +23,11 @@
     </link>
     <gazebo reference="laser_frame">
-        <sensor name="laser" type="ray">
+        <sensor name="laser" type="gpu_lidar">
             <pose>0 0 0 0 0 0</pose>
+            <always_on>true</always_on>
             <visualize>false</visualize>
             <update_rate>10</update_rate>
+            <topic>scan</topic>
+            <gz_frame_id>laser_frame</gz_frame_id>
             <ray>
                 <scan>
@@ -41,11 +44,4 @@
                 </range>
             </ray>
-            <plugin name="laser_controller" filename="libgazebo_ros_ray_sensor.so">
-                <ros>
-                    <argument>~/out:=scan</argument>
-                </ros>
-                <output_type>sensor_msgs/LaserScan</output_type>
-                <frame_name>laser_frame</frame_name>
-            </plugin>
         </sensor>
         <material>Gazebo/Red</material>

File: description/robot_core.xacro (robot description, xacro)
@@ -75,4 +75,5 @@
         <origin xyz="0 ${wheel_offset_y} 0" rpy="-${pi/2} 0 0"/>
         <axis xyz="0 0 1"/>
+        <limit effort="10.0" velocity="10.0"/>
     </joint>
     <link name="left_wheel">
@@ -101,4 +102,5 @@
         <origin xyz="0 ${-wheel_offset_y} 0" rpy="${pi/2} 0 0"/>
         <axis xyz="0 0 -1"/>
+        <limit effort="10.0" velocity="10.0"/>
     </joint>
     <link name="right_wheel">

File: description/ros2_control.xacro (robot description, xacro)
@@ -1,7 +1,7 @@
 <?xml version="1.0"?>
 <robot xmlns:xacro="http://www.ros.org/wiki/xacro">
-    <ros2_control name="GazeboSystem" type="system">
+    <ros2_control name="GazeboSimSystem" type="system">
         <hardware>
-            <plugin>gazebo_ros2_control/GazeboSystem</plugin>
+            <plugin>gz_ros2_control/GazeboSimSystem</plugin>
         </hardware>
         <joint name="left_wheel_joint">
@@ -11,5 +11,4 @@
             </command_interface>
             <state_interface name="velocity"/>
-            <state_interface name="position"/>
         </joint>
         <joint name="right_wheel_joint">
@@ -19,9 +18,8 @@
             </command_interface>
             <state_interface name="velocity"/>
-            <state_interface name="position"/>
         </joint>
     </ros2_control>
     <gazebo>
-        <plugin name="gazebo_ros2_control" filename="libgazebo_ros2_control.so">
+        <plugin name="gz_ros2_control::GazeboSimROS2ControlPlugin" filename="libgz_ros2_control-system.so">
             <parameters>$(find ar_project)/config/my_controllers.yaml</parameters>
         </plugin>

Commit message: Migrate sim navigation stack to RGB-D RTAB-Map

File: description/camera.xacro (robot description, xacro)
@@ -25,7 +25,7 @@
             <always_on>true</always_on>
             <visualize>true</visualize>
-            <update_rate>10</update_rate>
+            <update_rate>30</update_rate>
             <camera>
-                <camera_info_topic>camera/camera_info</camera_info_topic>
+                <camera_info_topic>camera/camera/color/camera_info</camera_info_topic>
                 <horizontal_fov>1.089</horizontal_fov>
                 <image>
@@ -39,5 +39,5 @@
                 </clip>
             </camera>
-            <topic>camera/image_raw</topic>
+            <topic>camera/camera/color/image_raw</topic>
             <gz_frame_id>camera_link_optical</gz_frame_id>
         </sensor>

File: description/depth_camera.xacro (robot description, xacro)
@@ -1,32 +1,31 @@
 <?xml version="1.0"?>
 <robot xmlns:xacro="http://www.ros.org/wiki/xacro">
+    <!--
+      Keep legacy depth_camera_* frames as aliases so existing code keeps
+      working, but mount the simulated depth sensor on the same physical
+      camera_link/camera_link_optical frames as the RGB camera.
+    -->
     <joint name="depth_camera_joint" type="fixed">
-        <parent link="chassis"/>
+        <parent link="camera_link"/>
         <child link="depth_camera_link"/>
-        <origin xyz="0.455 0 0.08" rpy="0 0 0"/>
+        <origin xyz="0 0 0" rpy="0 0 0"/>
     </joint>
-    <link name="depth_camera_link">
-        <visual>
-            <geometry>
-                <box size="0.01 0.03 0.03"/>
-            </geometry>
-            <material name="red"/>
-        </visual>
-    </link>
+    <link name="depth_camera_link"></link>
     <joint name="depth_camera_optical_joint" type="fixed">
-        <parent link="depth_camera_link"/>
+        <parent link="camera_link_optical"/>
         <child link="depth_camera_link_optical"/>
-        <origin xyz="0 0 0" rpy="${-pi/2} 0 ${-pi/2}"/>
+        <origin xyz="0 0 0" rpy="0 0 0"/>
     </joint>
     <link name="depth_camera_link_optical"></link>
-    <gazebo reference="depth_camera_link">
+    <gazebo reference="camera_link">
         <sensor name="depth_camera" type="depth">
             <pose>0 0 0 0 0 0</pose>
             <always_on>true</always_on>
             <visualize>true</visualize>
-            <update_rate>10</update_rate>
-            <topic>depth_camera/depth/image_raw</topic>
-            <gz_frame_id>depth_camera_link_optical</gz_frame_id>
+            <update_rate>30</update_rate>
+            <topic>camera/camera/depth/image_rect_raw</topic>
+            <gz_frame_id>camera_link_optical</gz_frame_id>
             <camera>
+                <camera_info_topic>camera/camera/depth/camera_info</camera_info_topic>
                 <horizontal_fov>1.089</horizontal_fov>
                 <image>
@@ -42,5 +41,4 @@
             </camera>
         </sensor>
-        <material>Gazebo/Red</material>
     </gazebo>
 </robot>

File: description/robot.urdf.xacro (robot description, xacro)
@@ -9,5 +9,4 @@
         <xacro:include filename="gazebo_control.xacro"/>
     </xacro:unless>
-    <xacro:include filename="lidar.xacro"/>
     <xacro:include filename="camera.xacro"/>
     <xacro:include filename="depth_camera.xacro"/>

Commit message: Refine embodied RGB-D navigation and camera description

File: description/camera.xacro (robot description, xacro)
@@ -4,10 +4,10 @@
         <parent link="chassis"/>
         <child link="camera_link"/>
-        <origin xyz="0.455 0 0.08" rpy="0 0 0"/>
+        <origin xyz="${camera_mount_x} 0 ${camera_mount_z}" rpy="0 0 0"/>
     </joint>
     <link name="camera_link">
         <visual>
             <geometry>
-                <box size="0.01 0.03 0.03"/>
+                <box size="0.025 0.09 0.025"/>
             </geometry>
             <material name="red"/>
@@ -20,27 +20,3 @@
     </joint>
     <link name="camera_link_optical"></link>
-    <gazebo reference="camera_link">
-        <sensor name="camera" type="camera">
-            <pose>0 0 0 0 0 0</pose>
-            <always_on>true</always_on>
-            <visualize>true</visualize>
-            <update_rate>30</update_rate>
-            <camera>
-                <camera_info_topic>camera/camera/color/camera_info</camera_info_topic>
-                <horizontal_fov>1.089</horizontal_fov>
-                <image>
-                    <format>R8G8B8</format>
-                    <width>640</width>
-                    <height>480</height>
-                </image>
-                <clip>
-                    <near>0.05</near>
-                    <far>8.0</far>
-                </clip>
-            </camera>
-            <topic>camera/camera/color/image_raw</topic>
-            <gz_frame_id>camera_link_optical</gz_frame_id>
-        </sensor>
-        <material>Gazebo/Red</material>
-    </gazebo>
 </robot>

File: description/depth_camera.xacro (robot description, xacro)
@@ -18,27 +18,3 @@
     </joint>
     <link name="depth_camera_link_optical"></link>
-    <gazebo reference="camera_link">
-        <sensor name="depth_camera" type="depth">
-            <pose>0 0 0 0 0 0</pose>
-            <always_on>true</always_on>
-            <visualize>true</visualize>
-            <update_rate>30</update_rate>
-            <topic>camera/camera/depth/image_rect_raw</topic>
-            <gz_frame_id>camera_link_optical</gz_frame_id>
-            <camera>
-                <camera_info_topic>camera/camera/depth/camera_info</camera_info_topic>
-                <horizontal_fov>1.089</horizontal_fov>
-                <image>
-                    <width>640</width>
-                    <height>480</height>
-                </image>
-                <depth_camera>
-                    <clip>
-                        <near>0.05</near>
-                        <far>8.0</far>
-                    </clip>
-                </depth_camera>
-            </camera>
-        </sensor>
-    </gazebo>
 </robot>

File: description/robot.urdf.xacro (robot description, xacro)
@@ -11,3 +11,4 @@
     <xacro:include filename="camera.xacro"/>
     <xacro:include filename="depth_camera.xacro"/>
+    <xacro:include filename="camera_gazebo_sensors.xacro"/>
 </robot>

File: description/robot_core.xacro (robot description, xacro)
@@ -2,18 +2,21 @@
 <robot xmlns:xacro="http://www.ros.org/wiki/xacro">
     <xacro:include filename="inertial_macros.xacro"/>
-    <xacro:property name="chassis_length" value="0.45"/>
-    <xacro:property name="chassis_width" value="0.3"/>
-    <xacro:property name="chassis_height" value="0.15"/>
     <xacro:property name="chassis_mass" value="0.7"/>
     <xacro:property name="wheel_radius" value="0.039"/>
-    <xacro:property name="wheel_thickness" value="0.04"/>
+    <xacro:property name="chassis_radius" value="0.12"/>
+    <xacro:property name="chassis_height" value="0.053"/>
+    <xacro:property name="chassis_bottom_from_floor" value="0.013"/>
+    <xacro:property name="chassis_center_z" value="${chassis_bottom_from_floor + chassis_height/2 - wheel_radius}"/>
+    <xacro:property name="wheel_thickness" value="0.018"/>
     <xacro:property name="wheel_mass" value="0.01"/>
-    <xacro:property name="wheel_offset_x" value="0.1"/>
+    <xacro:property name="wheel_offset_x" value="0.0"/>
     <xacro:property name="wheel_offset_y" value="0.1475"/>
     <xacro:property name="wheel_offset_z" value="0"/>
-    <xacro:property name="caster_wheel_radius" value="0.05"/>
+    <xacro:property name="caster_wheel_radius" value="0.015"/>
     <xacro:property name="caster_wheel_mass" value="0.25"/>
-    <xacro:property name="caster_wheel_offset_x" value="0.37"/>
+    <xacro:property name="caster_wheel_offset_x" value="0.09"/>
     <xacro:property name="caster_wheel_offset_z" value="${wheel_offset_z - wheel_radius + caster_wheel_radius}"/>
+    <xacro:property name="camera_mount_x" value="0.12"/>
+    <xacro:property name="camera_mount_z" value="0.0395"/>
     <material name="white">
         <color rgba="1 1 1 1"/>
@@ -38,5 +41,5 @@
         <parent link="base_link"/>
         <child link="base_footprint"/>
-        <origin xyz="0 0 0" rpy="0 0 0"/>
+        <origin xyz="0 0 -${wheel_radius}" rpy="0 0 0"/>
     </joint>
     <link name="base_footprint">
@@ -46,26 +49,27 @@
         <parent link="base_link"/>
         <child link="chassis"/>
-        <origin xyz="${-wheel_offset_x} 0 0"/>
+        <origin xyz="0 0 0"/>
     </joint>
     <link name="chassis">
         <visual>
-            <origin xyz="${chassis_length/2} 0 ${chassis_height/2}"/>
+            <origin xyz="0 0 ${chassis_center_z}"/>
             <geometry>
-                <box size="${chassis_length} ${chassis_width} ${chassis_height}"/>
+                <cylinder radius="${chassis_radius}" length="${chassis_height}"/>
             </geometry>
             <material name="white"/>
         </visual>
         <collision>
-            <origin xyz="${chassis_length/2} 0 ${chassis_height/2}"/>
+            <origin xyz="0 0 ${chassis_center_z}"/>
             <geometry>
-                <box size="${chassis_length} ${chassis_width} ${chassis_height}"/>
+                <cylinder radius="${chassis_radius}" length="${chassis_height}"/>
             </geometry>
         </collision>
-        <xacro:inertial_box mass="${chassis_mass}" x="${chassis_length}" y="${chassis_width}" z="${chassis_height}">
-            <origin xyz="${chassis_length/2} 0 ${chassis_height/2}" rpy="0 0 0"/>
-        </xacro:inertial_box>
+        <xacro:inertial_cylinder mass="${chassis_mass}" length="${chassis_height}" radius="${chassis_radius}">
+            <origin xyz="0 0 ${chassis_center_z}" rpy="0 0 0"/>
+        </xacro:inertial_cylinder>
     </link>
     <gazebo reference="chassis">
         <material>Gazebo/White</material>
+        <transparency>0.0</transparency>
     </gazebo>
     <!-- LEFT WHEEL LINK -->

File: description/robot_hardware.urdf.xacro (robot description, xacro)
@@ -4,3 +4,7 @@
     <xacro:include filename="robot_core.xacro"/>
     <xacro:include filename="ros2_control_hardware.xacro"/>
+    <!-- Keep the camera mount and legacy depth aliases in the real robot
+         description so the RealSense TF tree can attach to base_link. -->
+    <xacro:include filename="camera.xacro"/>
+    <xacro:include filename="depth_camera.xacro"/>
 </robot>
