Commit message: FLAT baseline fixes + VLM deployment docs
Keep the FLAT executive as the comparison baseline and land the sim fixes
verified across this work: nav2 transform_tolerance (RTAB-Map map->odom lag on
WSL2), caster sphere + wheel/chassis mass (in-place rotation), rsp ParameterValue
wrap, flat_sim_bringup params_file pin + gui passthrough. Executive tuning kept:
frontier degenerate-skip (skill_logic/skills), approach reacquire-distance,
seek_object await-detection + active_subtask feedback, prompt_bridge instruction
normalizer (FLAT path only -- the VLM path takes the raw label).

Update RUNBOOK + HIL checklist for the new VLM vocabulary, perception (distance +
SLAM map), params (async_replan / detect_conf / send_map / map_max_px /
vlm_timeout_s), the bare-label requirement, GZ_IP sim note, and the Pi/edge run
and mission-start steps.

File: ar_project/description/robot_core.xacro (robot description, xacro)
@@ -2,8 +2,11 @@
 <robot xmlns:xacro="http://www.ros.org/wiki/xacro">
     <xacro:include filename="inertial_macros.xacro"/>
-    <xacro:property name="chassis_mass" value="0.7"/>
+    <!-- Masses tuned for stable gz contact/traction. The original 0.01 kg wheels
+         gave tiny inertia (~5e-6) so the contact solver could rotate but not reliably
+         translate the body (wheels spun without gripping). Realistic values fix it. -->
+    <xacro:property name="chassis_mass" value="1.5"/>
     <xacro:property name="wheel_radius" value="0.038"/>
     <xacro:property name="wheel_thickness" value="0.033"/>
-    <xacro:property name="wheel_mass" value="0.01"/>
+    <xacro:property name="wheel_mass" value="0.25"/>
     <xacro:property name="chassis_length" value="0.36"/>
     <xacro:property name="chassis_width" value="0.30"/>
@@ -98,4 +101,6 @@
     <gazebo reference="left_wheel">
         <material>Gazebo/Blue</material>
+        <mu1>1.0</mu1>
+        <mu2>1.0</mu2>
     </gazebo>
     <!-- RIGHT WHEEL LINK -->
@@ -125,4 +130,6 @@
     <gazebo reference="right_wheel">
         <material>Gazebo/Blue</material>
+        <mu1>1.0</mu1>
+        <mu2>1.0</mu2>
     </gazebo>
     <!-- FRONT CENTER CASTER WHEEL LINK -->
@@ -140,6 +147,8 @@
         </visual>
         <collision>
+            <!-- Passive omni support modelled as a sphere - point contact slides freely
+                 in any direction (a fixed cylinder skids and blocks in-place rotation). -->
             <geometry>
-                <cylinder radius="${wheel_radius}" length="${wheel_thickness}"/>
+                <sphere radius="${wheel_radius}"/>
             </geometry>
         </collision>
@@ -150,4 +159,7 @@
     <gazebo reference="caster_wheel">
         <material>Gazebo/Blue</material>
+        <!-- Frictionless so the passive support never resists driving/turning. -->
+        <mu1>0.0</mu1>
+        <mu2>0.0</mu2>
     </gazebo>
 </robot>
